Commit message: rename package

File: urdf/only_servo.SLDASM.urdf (robot description, URDF)
Before this commit: robot only_servo.SLDASM, 3 links, 2 joints
Links:
- link camera_mount_link: geometry collision mesh filename=package://a1_neck_description/meshes/camera_mount_link.STL; visual mesh filename=package://a1_neck_description/meshes/camera_mount_link.STL
- link servo2_link: geometry collision mesh filename=package://a1_neck_description/meshes/servo2_link.STL; visual mesh filename=package://a1_neck_description/meshes/servo2_link.STL
- link stab_link: geometry collision mesh filename=package://a1_neck_description/meshes/stab_link.STL; visual mesh filename=package://a1_neck_description/meshes/stab_link.STL
