Commit message: del camera visual

File: urdf/neck.urdf.xacro (robot description, xacro)
@@ -5,4 +5,5 @@
 <robot name="a1_neck" xmlns:xacro="http://ros.org/wiki/xacro">
   <xacro:macro name="a1_neck" params="parent *origin">
+    <xacro:property name="M_PI" value="3.1415926535897931" />
     <!-- connect external origin with local root link -->
     <joint name="a1_neck_joint" type="fixed">
@@ -13,7 +14,5 @@
     <link name="stab_link">
       <inertial>
-        <origin
-          xyz="0.012635 0.0 0.0011677"
-          rpy="0 0 0" />
+        <origin xyz="0.012635 0.0 0.0011677" rpy="0 0 0" />
         <mass
           value="0.042672" />
@@ -108,44 +107,6 @@
         velocity="6" />
     </joint>
-    <link
-      name="camera_mount_link">
-      <inertial>
-        <origin
-          xyz="0.0015655 0.011821 0.005"
-          rpy="0 0 0" />
-        <mass
-          value="0.11501" />
-        <inertia
-          ixx="3.6446E-05"
-          ixy="1.0588E-22"
-          ixz="-1.38E-21"
-          iyy="6.5851E-06"
-          iyz="-1.2581E-21"
-          izz="4.1114E-05" />
-      </inertial>
-      <visual>
-        <origin
-          xyz="0 0 0"
-          rpy="0 0 0" />
-        <geometry>
-          <mesh
-            filename="package://a1_neck_description/meshes/camera_mount_link.STL" />
-        </geometry>
-        <material
-          name="">
-          <color
-            rgba="0.79216 0.81961 0.93333 1" />
-        </material>
-      </visual>
-      <collision>
-        <origin
-          xyz="0 0 0"
-          rpy="0 0 0" />
-        <geometry>
-          <mesh
-            filename="package://a1_neck_description/meshes/camera_mount_link.STL" />
-        </geometry>
-      </collision>
-    </link>
+    <!-- Dummy link to connect realsense xacro -->
+    <link name="camera_mount_link"/>
     <joint
       name="servo2_to_camera"

Commit message: edit collision, dynamic params

File: urdf/neck.urdf.xacro (robot description, xacro)
@@ -4,4 +4,6 @@
      For more information, please see http://wiki.ros.org/sw_urdf_exporter -->
 <robot name="a1_neck" xmlns:xacro="http://ros.org/wiki/xacro">
+    <xacro:property name="damping" value="3.121E-6"/>
+    <xacro:property name="friction" value="2.369E-4"/>
   <xacro:macro name="a1_neck" params="parent *origin">
     <!-- connect external origin with local root link -->
@@ -9,7 +11,7 @@
       <xacro:insert_block name="origin" />
       <parent link="${parent}"/>
-      <child link="stab_link" />
+      <child link="servo_link_1" />
     </joint>
-    <link name="stab_link">
+    <link name="servo_link_1">
       <inertial>
         <origin
@@ -32,5 +34,5 @@
         <geometry>
           <mesh
-            filename="package://a1_neck_description/meshes/stab_link.STL" />
+            filename="package://a1_neck_description/meshes/servo_link_1.STL" />
         </geometry>
         <material
@@ -42,14 +44,16 @@
       <collision>
         <origin
-          xyz="0 0 0"
+          xyz="0.013 0 0.002"
           rpy="0 0 0" />
-        <geometry>
-          <mesh
-            filename="package://a1_neck_description/meshes/stab_link.STL" />
-        </geometry>
+            <geometry>
+                <box size=".05 .028 .033"/>
+            </geometry>
+            <material name="">
+              <color rgba="1. 0. 0. 1" />
+            </material>
       </collision>
     </link>
     <link
-      name="servo2_link">
+      name="servo_link_2">
       <inertial>
         <origin
@@ -72,5 +76,5 @@
         <geometry>
           <mesh
-            filename="package://a1_neck_description/meshes/servo2_link.STL" />
+            filename="package://a1_neck_description/meshes/servo_link_2.STL" />
         </geometry>
         <material
@@ -82,10 +86,9 @@
       <collision>
         <origin
-          xyz="0 0 0"
+          xyz="0 0.016 0"
           rpy="0 0 0" />
-        <geometry>
-          <mesh
-            filename="package://a1_neck_description/meshes/servo2_link.STL" />
-        </geometry>
+            <geometry>
+                <box size=".055 .028 .033"/>
+            </geometry>
       </collision>
     </link>
@@ -95,9 +98,9 @@
       <origin
         xyz="0 -0.021 0"
-        rpy="-3.1416 -0.38051 0" />
+        rpy="-3.1416 0 0" />
       <parent
-        link="stab_link" />
+        link="servo_link_1" />
       <child
-        link="servo2_link" />
+        link="servo_link_2" />
       <axis
         xyz="0 1 0" />
@@ -107,45 +110,7 @@
         effort="10"
         velocity="6" />
+      <dynamics damping="${damping}" friction="${friction}"/>
     </joint>
-    <link
-      name="camera_mount_link">
-      <inertial>
-        <origin
-          xyz="0.0015655 0.011821 0.005"
-          rpy="0 0 0" />
-        <mass
-          value="0.11501" />
-        <inertia
-          ixx="3.6446E-05"
-          ixy="1.0588E-22"
-          ixz="-1.38E-21"
-          iyy="6.5851E-06"
-          iyz="-1.2581E-21"
-          izz="4.1114E-05" />
-      </inertial>
-      <visual>
-        <origin
-          xyz="0 0 0"
-          rpy="0 0 0" />
-        <geometry>
-          <mesh
-            filename="package://a1_neck_description/meshes/camera_mount_link.STL" />
-        </geometry>
-        <material
-          name="">
-          <color
-            rgba="0.79216 0.81961 0.93333 1" />
-        </material>
-      </visual>
-      <collision>
-        <origin
-          xyz="0 0 0"
-          rpy="0 0 0" />
-        <geometry>
-          <mesh
-            filename="package://a1_neck_description/meshes/camera_mount_link.STL" />
-        </geometry>
-      </collision>
-    </link>
+    <link name="camera_mount_link"/>
     <joint
       name="servo2_to_camera"
@@ -153,7 +118,7 @@
       <origin
         xyz="0 0.016 0.021"
-        rpy="0 0 1.7325" />
+        rpy="0 0 3.1415" />
       <parent
-        link="servo2_link" />
+        link="servo_link_2" />
       <child
         link="camera_mount_link" />
@@ -165,4 +130,5 @@
         effort="10"
         velocity="6" />
+      <dynamics damping="${damping}" friction="${friction}"/>
     </joint>
   </xacro:macro>
